File: Mechanical/PCB/Encoder/Stm32f072/_restore_backup_2026-09-06T22-18-40-535/Stm32f072.kicad_sch (KiCad schematic)
At the start: 41 parts, among them J1 Conn_01x04_Pin, U1 MP2451DT-LF-Z, U3 AS5047D, U4 STM32F072C8Tx, U5 SN65HVD230, Y1 Crystal

Commit message: fix sche, pcb layout
Parts:
- C10, C11, C12, C13, C14, C15, C4, C5, C6, C8, C9: footprint Capacitor_SMD:C_0603_1608Metric -> Capacitor_SMD:C_0603_1608Metric_Pad1.08x0.95mm_HandSolder
- CAN1, CAN2: footprint Connector_JST:JST_GH_BM04B-GHS-TBT_1x04-1MP_P1.25mm_Vertical -> Connector_JST:JST_XH_B4B-XH-A_1x04_P2.50mm_Vertical
- D_TVS1: footprint Diode_SMD:D_SMB -> Diode_SMD:D_SMB_Handsoldering
- J1: footprint Connector_Wire:SolderWire-0.127sqmm_1x04_P3.7mm_D0.48mm_OD1mm -> Connector_PinHeader_2.54mm:PinHeader_1x04_P2.54mm_Horizontal
- R1, R10, R2, R3, R5, R7, R8, R9: footprint Resistor_SMD:R_0603_1608Metric -> Resistor_SMD:R_0603_1608Metric_Pad0.98x0.95mm_HandSolder
- R6: footprint Resistor_SMD:R_0603_1608Metric -> Resistor_SMD:R_0805_2012Metric_Pad1.20x1.40mm_HandSolder
- U1: footprint Package_TO_SOT_SMD:SOT-23-6 -> Package_TO_SOT_SMD:SOT-23-6_Handsoldering
Other:
- moved on the sheet: JP1, R10, R5
