File: Mechanical/PCB/Encoder/Stm32f072/_restore_backup_2026-09-07T16-10-53-153/Stm32f072.kicad_pcb (KiCad board)
At the start: 2 copper layers, 42 x 42 mm, 41 parts, among them J1 Conn_01x04_Pin, U1 MP2451DT-LF-Z, U3 AS5047D, U4 STM32F072C8Tx, U5 SN65HVD230, Y1 Crystal

Commit message: fix sche, pcb layout
Parts:
- moved C12 36.0 mm to (141.4, 27.0), turned to 180 degrees
- moved JP3 33.2 mm to (148.3, 35.0)
- moved JP2 33.0 mm to (151.5, 35.0)
- moved C15 22.7 mm to (127.6, 35.0)
- moved C11 19.7 mm to (141.4, 35.0), turned to 180 degrees
- moved Debug1 1.93 mm to (152.0, 42.1)
- moved U5 0.15 mm to (150.8, 49.2)
Routing:
- net /CANL: track 18.4 -> 0.00 mm
- net /CANH: track 15.3 -> 0.00 mm
- net /MS1: track 10.1 -> 0.00 mm
- net /MS2: track 3.20 -> 0.00 mm
- net 3V3: track 9.57 -> 6.80 mm
Changed lines of the file:
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@@
 	(footprint "Capacitor_SMD:C_0603_1608Metric"
 		(layer "F.Cu")
-		(at 136.6 62.65)
+		(at 141.425 27 180)
 		(descr "Capacitor SMD 0603 (1608 Metric), square (rectangular) end terminal, IPC-7351 nominal, (Body size source: IPC-SM-782 page 76, https://www.pcb-3d.com/wordpress/wp-content/uploads/ipc-sm-782a_amendment_1_and_2.pdf)")
 		(tags "capacitor")
 		(property "Reference" "C12"
-			(at 0 -1.43 0)
+			(at 0 -1.43 180)
 			(layer "F.SilkS")
 			(effects
@@
 		)
 		(property "Value" "22pF"
-			(at 0 1.43 0)
+			(at 0 1.43 180)
 			(layer "F.Fab")
 			(effects
@@
 		)
 		(property "Datasheet" ""
-			(at 0 0 0)
+			(at 0 0 180)
 			(layer "F.Fab")
 			(hide yes)
@@
 		)
 		(property "Description" "Unpolarized capacitor"
-			(at 0 0 0)
+			(at 0 0 180)
 			(layer "F.Fab")
 			(hide yes)
@@
 		)
 		(property "KiLib_Generator" "SMD_2terminal_chip_molded"
-			(at 0 0 0)
+			(at 0 0 180)
 			(layer "F.SilkS")
 			(hide yes)
@@
 		(duplicate_pad_numbers_are_jumpers no)
 		(fp_line
-			(start -0.14058 -0.51)
-			(end 0.14058 -0.51)
+			(start -0.14058 0.51)
+			(end 0.14058 0.51)
 			(stroke
 				(width 0.12)
@@
 		)
 		(fp_line
-			(start -0.14058 0.51)
-			(end 0.14058 0.51)
+			(start -0.14058 -0.51)
+			(end 0.14058 -0.51)
 			(stroke
 				(width 0.12)
@@
 		)
 		(fp_text user "${REFERENCE}"
-			(at 0 0 0)
+			(at 0 0 180)
 			(layer "F.Fab")
 			(effects
@@
 		)
 		(pad "1" smd roundrect
-			(at -0.775 0)
+			(at -0.775 0 180)
 			(size 0.9 0.95)
 			(layers "F.Cu" "F.Mask" "F.Paste")
@@
 		)
 		(pad "2" smd roundrect
-			(at 0.775 0)
+			(at 0.775 0 180)
 			(size 0.9 0.95)
 			(layers "F.Cu" "F.Mask" "F.Paste")
@@
 	(footprint "Jumper:SolderJumper-3_P1.3mm_Open_Pad1.0x1.5mm_NumberLabels"
 		(layer "F.Cu")
-		(at 162.25 66.15 90)
+		(at 151.5 34.95 90)
 		(descr "SMD Solder Jumper, 1x1.5mm Pads, 0.3mm gap, open, labeled with numbers")
 		(tags "solder jumper open")
@@
 	(footprint "Capacitor_SMD:C_0603_1608Metric"
 		(layer "F.Cu")
-		(at 136.6 54.125)
+		(at 141.375 34.975 180)
 		(descr "Capacitor SMD 0603 (1608 Metric), square (rectangular) end terminal, IPC-7351 nominal, (Body size source: IPC-SM-782 page 76, https://www.pcb-3d.com/wordpress/wp-content/uploads/ipc-sm-782a_amendment_1_and_2.pdf)")
 		(tags "capacitor")
 		(property "Reference" "C11"
-			(at 0 -1.43 0)
+			(at 0 -1.43 180)
 			(layer "F.SilkS")
 			(effects
@@
 		)
 		(property "Value" "22pF"
-			(at 0 1.43 0)
+			(at 0 1.43 180)
 			(layer "F.Fab")
 			(effects
@@
 		)
 		(property "Datasheet" ""
-			(at 0 0 0)
+			(at 0 0 180)
 			(layer "F.Fab")
 			(hide yes)
@@
 		)
 		(property "Description" "Unpolarized capacitor"
-			(at 0 0 0)
+			(at 0 0 180)
 			(layer "F.Fab")
 			(hide yes)
@@
 		)
 		(property "KiLib_Generator" "SMD_2terminal_chip_molded"
-			(at 0 0 0)
+			(at 0 0 180)
 			(layer "F.SilkS")
 			(hide yes)
@@
 		(duplicate_pad_numbers_are_jumpers no)
 		(fp_line
-			(start -0.14058 -0.51)
-			(end 0.14058 -0.51)
+			(start -0.14058 0.51)
+			(end 0.14058 0.51)
 			(stroke
 				(width 0.12)
@@
 		)
 		(fp_line
-			(start -0.14058 0.51)
-			(end 0.14058 0.51)
+			(start -0.14058 -0.51)
+			(end 0.14058 -0.51)
 			(stroke
 				(width 0.12)
@@
 		)
 		(fp_text user "${REFERENCE}"
-			(at 0 0 0)
+			(at 0 0 180)
 			(layer "F.Fab")
 			(effects
@@
 		)
 		(pad "1" smd roundrect
-			(at -0.775 0)
+			(at -0.775 0 180)
 			(size 0.9 0.95)
 			(layers "F.Cu" "F.Mask" "F.Paste")
@@
 		)
 		(pad "2" smd roundrect
-			(at 0.775 0)
+			(at 0.775 0 180)
 			(size 0.9 0.95)
 			(layers "F.Cu" "F.Mask" "F.Paste")
@@
 	(footprint "Jumper:SolderJumper-3_P1.3mm_Open_Pad1.0x1.5mm_NumberLabels"
 		(layer "F.Cu")
-		(at 159.5 66.2 90)
+		(at 148.3 34.95 90)
 		(descr "SMD Solder Jumper, 1x1.5mm Pads, 0.3mm gap, open, labeled with numbers")
 		(tags "solder jumper open")
@@
 	(footprint "Connector_JST:JST_XH_B4B-XH-A_1x04_P2.50mm_Vertical"
 		(layer "F.Cu")
-		(at 150.1 42.275)
+		(at 152.025 42.125)
 		(descr "JST XH series connector, B4B-XH-A (http://www.jst-mfg.com/product/pdf/eng/eXH.pdf)")
 		(tags "connector JST XH vertical")
@@
 	(footprint "Package_SO:SOIC-8_3.9x4.9mm_P1.27mm"
 		(layer "F.Cu")
-		(at 150.8 49.1 180)
+		(at 150.825 49.25 180)
 		(descr "SOIC, 8 Pin (JEDEC MS-012AA, https://www.analog.com/media/en/package-pcb-resources/package/pkg_pdf/soic_narrow-r/r_8.pdf)")
 		(tags "SOIC SO")
@@
 	(footprint "Capacitor_SMD:C_0603_1608Metric"
 		(layer "F.Cu")
-		(at 139.8 54.125 180)
+		(at 127.6 35.025 180)
 		(descr "Capacitor SMD 0603 (1608 Metric), square (rectangular) end terminal, IPC-7351 nominal, (Body size source: IPC-SM-782 page 76, https://www.pcb-3d.com/wordpress/wp-content/uploads/ipc-sm-782a_amendment_1_and_2.pdf)")
 		(tags "capacitor")
@@
 	)
 	(segment
-		(start 159.55 67.45)
-		(end 159.5 67.5)
-		(width 0.2)
-		(layer "F.Cu")
-		(net "3V3")
-	)
-	(segment
 		(start 141.525 71.15)
 		(end 140.75 71.925)
@@
 	)
 	(segment
-		(start 162.25 67.45)
-		(end 159.55 67.45)
-		(width 0.2)
-		(layer "F.Cu")
-		(net "3V3")
-	)
-	(segment
 		(start 140.775 73.75)
 		(end 140.775 73.675)
@@
 	)
 	(segment
-		(start 163.3 66.65)
-		(end 163.3 68.5)
-		(width 0.2)
-		(layer "F.Cu")
-		(net "/MS1")
-	)
-	(segment
-		(start 157.79881 68.625)
-		(end 156.769405 67.595595)
-		(width 0.2)
-		(layer "F.Cu")
-		(net "/MS1")
-	)
-	(segment
-		(start 163.3 68.5)
-		(end 163.175 68.625)
-		(width 0.2)
-		(layer "F.Cu")
-		(net "/MS1")
-	)
-	(segment
-		(start 162.8 66.15)
-		(end 163.3 66.65)
-		(width 0.2)
-		(layer "F.Cu")
-		(net "/MS1")
-	)
-	(segment
-		(start 163.175 68.625)
-		(end 157.79881 68.625)
-		(width 0.2)
-		(layer "F.Cu")
-		(net "/MS1")
-	)
-	(segment
-		(start 162.25 66.15)
-		(end 162.8 66.15)
-		(width 0.2)
-		(layer "F.Cu")
-		(net "/MS1")
-	)
-	(segment
-		(start 141.775 42.9)
-		(end 141.525 43.15)
-		(width 0.2)
-		(layer "F.Cu")
-		(net "/CANL")
-	)
-	(segment
-		(start 148.35 48.615)
-		(end 148.004448 48.615)
-		(width 0.2)
-		(layer "F.Cu")
-		(net "/CANL")
-	)
-	(segment
-		(start 141.525 51.3)
-		(end 141.575 51.35)
-		(width 0.2)
-		(layer "F.Cu")
-		(net "/CANL")
-	)
-	(segment
-		(start 141.525 43.15)
-		(end 141.525 44.7)
-		(width 0.2)
-		(layer "F.Cu")
-		(net "/CANL")
-	)
-	(segment
-		(start 143.715552 42.9)
-		(end 141.775 42.9)
-		(width 0.2)
-		(layer "F.Cu")
-		(net "/CANL")
-	)
-	(segment
-		(start 141.525 44.7)
-		(end 141.525 51.3)
-		(width 0.2)
-		(layer "F.Cu")
-		(net "/CANL")
-	)
-	(segment
-		(start 146.725 45.909448)
-		(end 143.715552 42.9)
-		(width 0.2)
-		(layer "F.Cu")
-		(net "/CANL")
-	)
-	(segment
-		(start 148.004448 48.615)
-		(end 146.725 47.335552)
-		(width 0.2)
-		(layer "F.Cu")
-		(net "/CANL")
-	)
-	(segment
-		(start 146.725 47.335552)
-		(end 146.725 45.909448)
-		(width 0.2)
-		(layer "F.Cu")
-		(net "/CANL")
-	)
-	(segment
-		(start 144.060001 53.2)
-		(end 143.05 53.2)
-		(width 0.2)
-		(layer "F.Cu")
-		(net "/CANH")
-	)
-	(segment
-		(start 142.775 44.7)
-		(end 142.775 51.3)
-		(width 0.2)
-		(layer "F.Cu")
-		(net "/CANH")
-	)
-	(segment
-		(start 143.05 53.2)
-		(end 142.825 52.975)
-		(width 0.2)
-		(layer "F.Cu")
-		(net "/CANH")
-	)
-	(segment
-		(start 142.825 52.975)
-		(end 142.825 51.35)
-		(width 0.2)
-		(layer "F.Cu")
-		(net "/CANH")
-	)
-	(segment
-		(start 142.775 51.3)
-		(end 142.825 51.35)
-		(width 0.2)
-		(layer "F.Cu")
-		(net "/CANH")
-	)
-	(segment
-		(start 147.375001 49.885)
-		(end 144.060001 53.2)
-		(width 0.2)
-		(layer "F.Cu")
-		(net "/CANH")
-	)
-	(segment
-		(start 148.35 49.885)
-		(end 147.375001 49.885)
-		(width 0.2)
-		(layer "F.Cu")
-		(net "/CANH")
-	)
-	(segment
 		(start 152.65 77.55)
 		(end 152.75 77.45)
@@
 	)
 	(segment
-		(start 159.5 66.2)
-		(end 157.91381 66.2)
-		(width 0.2)
-		(layer "F.Cu")
-		(net "/MS2")
-	)
-	(segment
-		(start 157.91381 66.2)
-		(end 156.769405 65.055595)
-		(width 0.2)
-		(layer "F.Cu")
-		(net "/MS2")
-	)
-	(segment
