File: Mechanical/PCB/Encoder/FOC_Board/FOC_Board.kicad_pcb (KiCad board)
At the start: 4 copper layers, 60 x 60 mm, 91 parts, among them IC2 TPS563200DDCR, J1 CAN_IN, J2 CAN_OUT, J3 XT30PW-M, J4 U, J5 V, J6 W, J7 SWD, J8 UART, J9 HALL, Q1 CSD88537ND, Q2 CSD88537ND, Q3 CSD88537ND, U1 DRV8353RSRGZT, U2 STM32G431CBUx, U4 ME6211C33M5, U5 TJA1051T-3, Y2 8MHz

Commit message: layoutt
Routing:
- net ENC_SCK: track 0.00 -> 24.5 mm, vias 0 -> 2
- net ENC_MISO: track 0.00 -> 23.4 mm, vias 0 -> 2
- net ENC_CS: track 0.00 -> 22.1 mm, vias 0 -> 2
- net /MCU/DEBUG_CLK: track 0.00 -> 19.3 mm, vias 0 -> 2
- net /MCU/DEBUG_DIO: track 0.00 -> 19.2 mm, vias 0 -> 2
- net Net-(U2-PF1): track 0.00 -> 6.78 mm
- net Net-(U2-PF0): track 0.00 -> 5.90 mm
