File: Mechanical/PCB/Encoder/FOC_Board/FOC_Board.kicad_pcb (KiCad board)
At the start: 4 copper layers, 60 x 80 mm, 87 parts, among them IC2 TPS563200DDCR, J1 CAN_IN, J2 CAN_OUT, J7 SWD, J8 UART, Q1 CSD88537ND, Q2 CSD88537ND, Q3 CSD88537ND, U1 DRV8353RSRGZT, U2 STM32G431CBUx, U4 ME6211C33M5, U5 TJA1051T-3, Y1 8MHz

Commit message: add pcb, fix sche
Parts:
- removed Y1: 8MHz, Crystal:Crystal_SMD_5032-2Pin_5.0x3.2mm
- added J3: XT30PW-M, XT30PW-M:AMASS_XT30PW-M, F.Cu at (54.1, 86.0)
- added J4: U, Connector_Wire:SolderWire-1.5sqmm_1x01_D1.7mm_OD3mm, F.Cu at (158.4, 63.9)
- added J5: V, Connector_Wire:SolderWire-1.5sqmm_1x01_D1.7mm_OD3mm, F.Cu at (158.4, 69.1)
- added J6: W, Connector_Wire:SolderWire-1.5sqmm_1x01_D1.7mm_OD3mm, F.Cu at (158.4, 74.3)
- added J9: HALL, Connector_JST:JST_GH_BM06B-GHS-TBT_1x06-1MP_P1.25mm_Vertical, F.Cu at (169.7, 65.2)
- added Y2: 8MHz, Crystal:Crystal_SMD_3225-4Pin_3.2x2.5mm, F.Cu at (60.2, 65.7)
- moved C2 79.5 mm to (54.7, 67.0), turned to 90 degrees
- moved U2 76.6 mm to (66.8, 66.2)
- moved U1 72.7 mm to (79.2, 82.4)
- moved C1 72.5 mm to (61.0, 68.4)
- moved J1 66.2 mm to (105.8, 73.4), turned to 90 degrees
- moved J2 65.9 mm to (105.8, 63.5), turned to 90 degrees
- moved Q1 55.3 mm to (72.7, 93.1), turned to -90 degrees
- moved U5 55.1 mm to (93.6, 68.4)
- moved Q2 47.0 mm to (81.9, 93.1), turned to -90 degrees
- moved J8 45.0 mm to (84.0, 54.1), turned to 180 degrees
- moved Q3 39.1 mm to (92.2, 93.1), turned to -90 degrees
- moved J7 31.2 mm to (96.5, 54.1), turned to 180 degrees
- moved D6 10.2 mm to (132.3, 120.1)
- moved L1 10.2 mm to (131.2, 113.9)
- moved R5 10.2 mm to (147.4, 86.1)
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Connections:
- net /MCU/PWM_A+ renamed PWM_A+
- net /MCU/PWM_A- renamed PWM_A-
- net /MCU/PWM_B+ renamed PWM_B+
- net /MCU/PWM_B- renamed PWM_B-
- net /MCU/PWM_C+ renamed PWM_C+
- net /MCU/PWM_C- renamed PWM_C-
- net /MCU/VBUS_SENSED renamed VBUS_SENSED
- net /Three_phase/INHA renamed INHA
- net /Three_phase/INHB renamed INHB
- net /Three_phase/INHC renamed INHC
- net /Three_phase/INLA renamed INLA
- net /Three_phase/INLB renamed INLB
- net /Three_phase/INLC renamed INLC
- net /Three_phase/SHA renamed U
- net /Three_phase/SHB renamed V
- net /Three_phase/SHC renamed W
- net /Three_phase/V_BUS renamed V_BUS
- C13 pad 1: /MCU/3V3 -> 3V3
- C14 pad 1: /MCU/3V3 -> 3V3
- C3 pad 1: /Three_phase/PWR_GND -> GND
- C33 pad 2: /Three_phase/Buck -> 12V
- C35 pad 1: /Three_phase/PWR_GND -> GND
- C35 pad 2: /Three_phase/Buck -> 12V
- C36 pad 1: /Three_phase/PWR_GND -> GND
- C36 pad 2: /Three_phase/Buck -> 12V
- C4 pad 1: /Three_phase/PWR_GND -> GND
- C44 pad 1: /Three_phase/PWR_GND -> GND
- C45 pad 1: /Three_phase/PWR_GND -> GND
- C46 pad 1: /Three_phase/PWR_GND -> GND
- C5 pad 1: /Three_phase/PWR_GND -> GND
- C6 pad 1: /Three_phase/PWR_GND -> GND
- C6 pad 2: /Three_phase/3V3 -> 3V3
- C74 pad 1: /MCU/12V -> 12V
- C75 pad 1: /MCU/12V -> 12V
- C76 pad 1: /MCU/12V -> 12V
- D6 pad 2: /Three_phase/Buck -> 12V
- FB1 pad 1: /MCU/3V3 -> 3V3
- IC2 pad 3: /MCU/12V -> 12V
- J7 pad 1: /MCU/3V3 -> 3V3
- L1 pad 2: /Three_phase/Buck -> 12V
- R1 pad 1: /Three_phase/PWR_GND -> GND
- R1 pad 2: /Three_phase/DRV_EN -> DRV_EN
- R16 pad 1: /Three_phase/PWR_GND -> GND
- R17 pad 2: /Three_phase/Buck -> 12V
- R2 pad 1: /Three_phase/PWR_GND -> GND
- R27 pad 2: /MCU/3V3 -> 3V3
- R4 pad 1: /Three_phase/DRV_FAULT -> DRV_FAULT
- R4 pad 2: /Three_phase/3V3 -> 3V3
- SHUNT1 pad 2: /Three_phase/PWR_GND -> GND
- SHUNT2 pad 2: /Three_phase/PWR_GND -> GND
- SHUNT3 pad 2: /Three_phase/PWR_GND -> GND
- U1 pad 1: /Three_phase/PWR_GND -> GND
- U1 pad 12: /Three_phase/PWR_GND -> GND
- U1 pad 13: /Three_phase/PWR_GND -> GND
- U1 pad 22: /Three_phase/PWR_GND -> GND
- U1 pad 23: /Three_phase/IC -> IC
- U1 pad 24: /Three_phase/IB -> IB
- U1 pad 25: /Three_phase/IA -> IA
- U1 pad 26: /Three_phase/3V3 -> 3V3
- U1 pad 27: /Three_phase/PWR_GND -> GND
- U1 pad 28: /Three_phase/DRV_FAULT -> DRV_FAULT
- U1 pad 29: /Three_phase/DRV_MISO -> DRV_MISO
- U1 pad 30: /Three_phase/DRV_MOSI -> DRV_MOSI
- U1 pad 31: /Three_phase/DRV_SCK -> DRV_SCK
- U1 pad 32: /Three_phase/DRV_CS -> DRV_CS
- U1 pad 33: /Three_phase/DRV_EN -> DRV_EN
- U1 pad 41: /Three_phase/PWR_GND -> GND
- U1 pad 49: /Three_phase/PWR_GND -> GND
- U2 pad 10: /MCU/IA -> IA
- U2 pad 11: /MCU/IB -> IB
- U2 pad 12: /MCU/DRV_CS -> DRV_CS
- U2 pad 13: /MCU/DRV_SCK -> DRV_SCK
- U2 pad 14: /MCU/DRV_MISO -> DRV_MISO
- U2 pad 15: /MCU/SPI1_MOSI -> DRV_MOSI
- U2 pad 18: /MCU/IC -> IC
- U2 pad 19: /MCU/DRV_EN -> DRV_EN
- U2 pad 22: /MCU/DRV_FAULT -> DRV_FAULT
- U2 pad 38: /MCU/ENC_CS -> ENC_CS
- U2 pad 39: /MCU/ENC_SCK -> ENC_SCK
- U2 pad 40: /MCU/ENC_MISO -> ENC_MISO
- U2 pad 43: /MCU/ENC_MOSI -> ENC_MOSI
- U5 pad 1: /MCU/CAN_TX -> /MCU/FDCAN1_RX
- U5 pad 4: /MCU/CAN_RX -> /MCU/FDCAN1_TX
Routing:
- net GND: vias 0 -> 4
- net (no net): vias 4 -> 0
- added copper zone on In1.Cu, net GND

Commit message: layout
Parts:
- removed FB1: FerriteBead_Small, Inductor_SMD:L_0603_1608Metric_Pad1.05x0.95mm_HandSolder
- moved J9 104.1 mm to (66.1, 54.1), turned to 180 degrees
- moved J4 99.9 mm to (66.5, 103.2)
- moved J5 88.1 mm to (77.2, 103.2)
- moved R16 85.3 mm to (103.0, 36.1)
- moved C22 85.1 mm to (46.2, 76.8), turned to 90 degrees
- moved C23 84.4 mm to (48.2, 76.8), turned to 90 degrees
- moved C12 81.6 mm to (46.7, 81.0), turned to 180 degrees
- moved R14 81.0 mm to (108.7, 33.9), turned to -90 degrees
- moved R17 80.8 mm to (127.8, 43.4)
- moved C11 79.7 mm to (46.7, 83.5), turned to 180 degrees
- moved C34 79.2 mm to (107.5, 21.4)
- moved C35 79.2 mm to (107.5, 24.4)
- moved C33 79.2 mm to (107.5, 18.4)
- moved C36 79.2 mm to (107.5, 27.4)
- moved L1 79.2 mm to (114.7, 36.4)
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Connections:
- C15 pad 1: /MCU/3V3_MCU -> 3V3
- C16 pad 1: /MCU/3V3_MCU -> 3V3
- C17 pad 1: /MCU/3V3_MCU -> 3V3
- C18 pad 1: /MCU/3V3_MCU -> 3V3
- FB2 pad 1: /MCU/3V3_MCU -> 3V3
- JP2 pad 1: /MCU/3V3_MCU -> 3V3
- R10 pad 2: /MCU/3V3_MCU -> 3V3
- R11 pad 2: /MCU/3V3_MCU -> 3V3
- R12 pad 2: /MCU/3V3_MCU -> 3V3
- R5 pad 1: /MCU/3V3_MCU -> 3V3
- TH1 pad 2: /MCU/3V3_MCU -> 3V3
- U1 pad 34: INHA -> PWM_A+
- U1 pad 35: INLA -> PWM_A-
- U1 pad 36: INHB -> PWM_B+
- U1 pad 37: INLB -> PWM_B-
- U1 pad 38: INLC -> PWM_C-
- U1 pad 39: INHC -> PWM_C+
- U2 pad 1: /MCU/3V3_MCU -> 3V3
- U2 pad 23: /MCU/3V3_MCU -> 3V3
- U2 pad 35: /MCU/3V3_MCU -> 3V3
- U2 pad 48: /MCU/3V3_MCU -> 3V3
Routing:
- net /Three_phase/GLC: track 0.00 -> 34.9 mm, vias 0 -> 2
- net /Three_phase/GHC: track 0.00 -> 32.5 mm, vias 0 -> 2
- net U: track 0.00 -> 30.6 mm, vias 0 -> 1
- net /Three_phase/GHA: track 0.00 -> 29.7 mm, vias 0 -> 2
- net W: track 0.00 -> 27.7 mm, vias 0 -> 1
- net /Three_phase/GLA: track 0.00 -> 27.4 mm, vias 0 -> 2
- net /Three_phase/GLB: track 0.00 -> 27.1 mm, vias 0 -> 2
- net /Three_phase/GHB: track 0.00 -> 24.5 mm, vias 0 -> 2
- net V: track 0.00 -> 22.9 mm, vias 0 -> 1
- net /Three_phase/SPC: track 0.00 -> 17.1 mm, vias 0 -> 12
- net /Three_phase/SPA: track 0.00 -> 11.4 mm, vias 0 -> 8
- net /Three_phase/SPB: track 0.00 -> 10.5 mm, vias 0 -> 8
- added copper zone on B.Cu, net /Three_phase/SPA
- added copper zone on B.Cu, net /Three_phase/SPB
- added copper zone on B.Cu, net /Three_phase/SPC
- added copper zone on F.Cu, net GND
- added copper zone on F.Cu, net U
- added copper zone on F.Cu, net V
- added copper zone on F.Cu, net V_BUS
- added copper zone on F.Cu, net W
Other:
- board size 60 x 80 mm -> 60 x 60 mm

Commit message: push win
Parts:
- moved C76 117.3 mm to (51.6, 78.1), turned to -90 degrees
- moved L2 116.4 mm to (54.5, 71.2), turned to 90 degrees
- moved R85 115.9 mm to (51.6, 82.9), turned to 90 degrees
- moved C74 114.2 mm to (59.1, 80.6), turned to -90 degrees
- moved IC2 113.5 mm to (54.4, 78.5), turned to -90 degrees
- moved R84 113.4 mm to (53.4, 82.9), turned to -90 degrees
- moved R82 110.8 mm to (55.3, 83.0), turned to -90 degrees
- moved C75 110.8 mm to (61.6, 80.6), turned to -90 degrees
- moved C77 109.6 mm to (57.1, 79.0), turned to 90 degrees
- moved C78 108.4 mm to (73.0, 81.1)
- moved C79 108.4 mm to (73.0, 76.5)
- moved R83 108.3 mm to (57.1, 82.9), turned to 90 degrees
- moved R17 80.2 mm to (59.2, 85.0), turned to -90 degrees
- moved C33 79.4 mm to (64.2, 85.0), turned to 90 degrees
- moved C34 78.4 mm to (61.7, 85.0), turned to -90 degrees
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Connections:
- U1 pad 43: unconnected-(U1-VIN-Pad43) -> V_BUS
Routing:
- net GND: vias 4 -> 9
- net /Three_phase/SPA: vias 8 -> 3
