File: Mechanical/PCB/Encoder/FOC_Board/threephase.kicad_sch (KiCad schematic)
At the start: 34 parts, among them Q1 CSD88537ND, Q2 CSD88537ND, Q3 CSD88537ND, U1 DRV8353RSRGZT

Commit message: fix schematic
Parts:
- Q1, Q2, Q3: footprint SOIC127P600X175-8N -> CSD88537ND:SOIC127P600X175-8N
- renumbered SHUNT to SHUNT3

Commit message: add pcb, fix sche
Parts:
- added J4: U, Connector_Wire:SolderWire-1.5sqmm_1x01_D1.7mm_OD3mm, symbol Connector:Conn_01x01_Pin
- added J5: V, Connector_Wire:SolderWire-1.5sqmm_1x01_D1.7mm_OD3mm, symbol Connector:Conn_01x01_Pin
- added J6: W, Connector_Wire:SolderWire-1.5sqmm_1x01_D1.7mm_OD3mm, symbol Connector:Conn_01x01_Pin
Connections:
- net U: now also J4.1 (Pin_1)
- net V: now also J5.1 (Pin_1)
- net W: now also J6.1 (Pin_1)

Commit message: layout
Connections:
- net INHA renamed PWM_A+
- net INHB renamed PWM_B+
- net INHC renamed PWM_C+
- net INLA renamed PWM_A-
- net INLB renamed PWM_B-
- net INLC renamed PWM_C-
Changed lines of the file:
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@@
 		)
 	)
-	(global_label "INHB"
+	(global_label "PWM_B+"
 		(shape input)
 		(at 69.85 57.15 180)
@@
 		)
 		(property "Intersheetrefs" "${INTERSHEET_REFS}"
-			(at 62.329 57.15 0)
+			(at 58.882 57.15 0)
 			(hide yes)
 			(show_name no)
@@
 		)
 	)
-	(global_label "INLA"
+	(global_label "PWM_A-"
 		(shape input)
 		(at 69.85 52.07 180)
@@
 		)
 		(property "Intersheetrefs" "${INTERSHEET_REFS}"
-			(at 62.8128 52.07 0)
+			(at 59.0634 52.07 0)
 			(hide yes)
 			(show_name no)
@@
 		)
 	)
-	(global_label "INLB"
+	(global_label "PWM_B-"
 		(shape input)
 		(at 69.85 59.69 180)
@@
 		)
 		(property "Intersheetrefs" "${INTERSHEET_REFS}"
-			(at 62.6314 59.69 0)
+			(at 58.882 59.69 0)
 			(hide yes)
 			(show_name no)
@@
 		)
 	)
-	(global_label "INHA"
+	(global_label "PWM_A+"
 		(shape input)
 		(at 69.85 49.53 180)
@@
 		)
 		(property "Intersheetrefs" "${INTERSHEET_REFS}"
-			(at 62.5104 49.53 0)
+			(at 59.0634 49.53 0)
 			(hide yes)
 			(show_name no)
@@
 		)
 	)
-	(global_label "INHC"
+	(global_label "PWM_C+"
 		(shape input)
 		(at 69.85 64.77 180)
@@
 		)
 		(property "Intersheetrefs" "${INTERSHEET_REFS}"
-			(at 62.329 64.77 0)
+			(at 58.882 64.77 0)
 			(hide yes)
 			(show_name no)
@@
 		)
 	)
-	(global_label "INLC"
+	(global_label "PWM_C-"
 		(shape input)
 		(at 69.85 67.31 180)
@@
 		)
 		(property "Intersheetrefs" "${INTERSHEET_REFS}"
-			(at 62.6314 67.31 0)
-			(hide yes)
-			(show_name no)
+			(at 58.882 67.31 0)
+			(hide yes)
+			(show_name no)

Commit message: push win
Connections:
- net V_BUS: now also U1.43 (VIN)
Changed lines of the file:
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@@
+	)
+	(junction
+		(at 66.04 34.29)
+		(diameter 0)
+		(color 0 0 0 0)
 	)
 	(junction
@@
 		)
 		(stroke
+			(width 0)
+			(type default)
+		)
+	)
+	(wire
+		(pts
+			(xy 66.04 34.29) (xy 73.66 34.29)
+		)
+		(stroke
