File: Mechanical/PCB/Encoder/FOC_Board/mcu.kicad_sch (KiCad schematic)
At the start: 54 parts, among them IC2 TPS563200DDCR, J1 Conn_01x01_Pin, J2 Conn_01x01_Pin, J7 SWD, J8 UART, J9 Conn_01x01_Pin, U2 STM32G431CBUx, U4 ME6211C33M5, U5 TJA1051T-3, Y1 8MHz

Commit message: fix schematic
Parts:
- removed J1, J2, J9: Conn_01x01_Pin, Connector_Wire:SolderWirePad_1x01_SMD_2x4mm, symbol Connector:Conn_01x01_Pin
- added J1: CAN_IN, Connector_JST:JST_GH_BM04B-GHS-TBT_1x04-1MP_P1.25mm_Vertical, symbol Connector:Conn_01x04_Pin
- added J2: CAN_OUT, Connector_JST:JST_GH_BM04B-GHS-TBT_1x04-1MP_P1.25mm_Vertical, symbol Connector:Conn_01x04_Pin
- C1, C2: footprint (none) -> Capacitor_SMD:C_0402_1005Metric
- J7, J8: footprint Connector_JST:JST_XH_B4B-XH-A_1x04_P2.50mm_Vertical -> Connector_JST:JST_GH_BM04B-GHS-TBT_1x04-1MP_P1.25mm_Vertical
Connections:
- net CANH: now also J1.3 (Pin_3), J2.3 (Pin_3)
- net CANL: now also J1.2 (Pin_2), J2.2 (Pin_2)
- net GND: now also J1.1 (Pin_1), J1.4 (Pin_4), J2.1 (Pin_1), J2.4 (Pin_4)

Commit message: add pcb, fix sche
Parts:
- removed Y1: 8MHz, Crystal:Crystal_SMD_5032-2Pin_5.0x3.2mm, symbol Device:Crystal
- added J3: XT30PW-M, XT30PW-M:AMASS_XT30PW-M, symbol XT30PW-M:XT30PW-M
- added J9: HALL, Connector_JST:JST_GH_BM06B-GHS-TBT_1x06-1MP_P1.25mm_Vertical, symbol Connector:Conn_01x06_Pin
- added Y2: 8MHz, Crystal:Crystal_SMD_3225-4Pin_3.2x2.5mm, symbol Device:Crystal_GND24_Small
Connections:
- net CAN_RX is gone; now on net FDCAN1_TX: U5.4 (RXD)
- net CAN_TX is gone; now on net FDCAN1_RX: U5.1 (TXD)
- net +5V: now also J9.6 (Pin_6)
- net ENC_CS: now also J9.2 (Pin_2)
- net ENC_MISO: now also J9.4 (Pin_4)
- net ENC_MOSI: now also J9.3 (Pin_3)
- net ENC_SCK: now also J9.5 (Pin_5)
- net GND: now also J3.N, J9.1 (Pin_1), Y2.2 (G), Y2.4 (G)
- net at C1.2, U2.6 (PF1): now also Y2.3
- net at C2.2, U2.5 (PF0): now also Y2.1
- new net V_BUS: J3.P
Other:
- moved on the sheet: C1, C2

Commit message: layout
Parts:
- removed FB1: FerriteBead_Small, Inductor_SMD:L_0603_1608Metric_Pad1.05x0.95mm_HandSolder, symbol Device:FerriteBead_Small
Connections:
- net 3V3_MCU is gone; now on net 3V3: C15.1, C16.1, C17.1, C18.1, FB2.1, JP2.1 (A), R10.2, R11.2, R12.2, R5.1, TH1.2, U2.1 (VBAT), U2.23 (VDD), U2.35 (VDD), U2.48 (VDD)
Other:
- moved on the sheet: C19, C20, FB2

Commit message: OPEN LOOP FOC
Other:
- note added: "ANALOG POWER"
- note added: "LED"
- note added: "MCU"
- note added: "POWER"
- moved on the sheet: C1, C13, C14, C15, C16, C17, C18, C19, C2, C20, C57, C58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
