File: Mechanical/PCB/Encoder/Stm32f072/Stm32f072.kicad_pcb (KiCad board)
At the start: 2 copper layers, 42 x 42 mm, 41 parts, among them J1 Conn_01x04_Pin, U1 MP2451DT-LF-Z, U3 AS5047D, U4 STM32F072C8Tx, U5 SN65HVD230, Y1 Crystal

Commit message: layoutt
Parts:
- R6: moved to F.Cu
- moved R9 56.1 mm to (164.4, 66.6)
- moved C14 36.4 mm to (150.4, 54.1), turned to 0 degrees
- moved D3 34.5 mm to (131.9, 54.8), turned to 180 degrees
- moved R8 34.4 mm to (131.5, 56.7)
- moved R10 34.1 mm to (131.5, 58.4), turned to 180 degrees
- moved R6 33.6 mm to (148.7, 52.6), turned to 0 degrees
- moved JP1 28.6 mm to (131.7, 50.7)
- moved C13 28.3 mm to (131.5, 52.9), turned to 0 degrees
- moved R5 23.9 mm to (131.5, 48.6), turned to 180 degrees
- moved C10 7.38 mm to (150.8, 65.1)
- moved C9 7.38 mm to (150.8, 66.8)
- moved D2 2.81 mm to (138.2, 75.7)
Routing:
- net 3V3: track 9.57 -> 143.6 mm, vias 0 -> 3
- net /EN: track 0.00 -> 29.1 mm
- net /PA9: track 0.00 -> 20.0 mm, vias 0 -> 1
- net /SWDIO: track 0.00 -> 18.7 mm, vias 0 -> 1
- net /BOOT0: track 0.00 -> 16.2 mm
- net /NRST: track 0.00 -> 15.1 mm
- net /SWCLK: track 0.00 -> 14.4 mm, vias 0 -> 1
- net /CAN_RX: track 0.00 -> 13.3 mm
- net /PC13: track 0.00 -> 12.5 mm
- net /PB13: track 0.00 -> 10.5 mm
- net /DIR: track 0.00 -> 10.4 mm
- net /MOSI: track 0.00 -> 9.96 mm, vias 0 -> 1
- net /CAN_TX: track 0.00 -> 9.54 mm
- net /CLK: track 0.00 -> 9.45 mm, vias 0 -> 1
- net /CS: track 0.00 -> 9.12 mm, vias 0 -> 1
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